File: schematics/VOLF_enhanced_transmitter/VOLF_enhanced_transmitter.kicad_sch (KiCad schematic)
At the start: 9 parts, among them J2 MCU DP2, J3 MCU GND

Commit message: added documentation for passive circuits
Parts:
- gave numbers to parts that had none: 1
Changed lines of the file:
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@@
 		(dnp no)
 		(fields_autoplaced yes)
-		(property "Reference" "C?"
+		(property "Reference" "C1"
 			(at 96.0881 60.96 0)
 			(effects
@@
 				)
 				(justify left)
-				(hide yes)
 			)
 		)
@@
 			(project "VOLK_enhanced_transmitter"
 				(path "/18397c79-8016-4b55-8616-aabd5bfb4047"
-					(reference "C?")
+					(reference "C1")
 					(unit 1)
 				)

Commit message: updated schematics
Parts:
- gave numbers to parts that had none: 6
Changed lines of the file:
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@@
 		(dnp no)
 		(fields_autoplaced yes)
-		(property "Reference" "R?"
+		(property "Reference" "R1"
 			(at 105.41 53.3399 0)
 			(effects
@@
 			(project "VOLK_enhanced_transmitter"
 				(path "/18397c79-8016-4b55-8616-aabd5bfb4047"
-					(reference "R?")
+					(reference "R1")
 					(unit 1)
 				)
@@
 		(on_board yes)
 		(dnp no)
-		(fields_autoplaced yes)
-		(property "Reference" "J?"
-			(at 83.185 74.93 0)
-			(effects
-				(font
-					(size 1.27 1.27)
-				)
+		(property "Reference" "J1"
+			(at 86.106 74.93 0)
+			(effects
+				(font
+					(size 1.27 1.27)
+				)
+				(justify right)
 			)
 		)
 		(property "Value" "AudioJack3"
-			(at 83.185 72.39 0)
-			(effects
-				(font
-					(size 1.27 1.27)
-				)
+			(at 89.662 72.39 0)
+			(effects
+				(font
+					(size 1.27 1.27)
+				)
+				(justify right)
 			)
 		)
@@
 			(project "VOLK_enhanced_transmitter"
 				(path "/18397c79-8016-4b55-8616-aabd5bfb4047"
-					(reference "J?")
+					(reference "J1")
 					(unit 1)
 				)
@@
 		(dnp no)
 		(fields_autoplaced yes)
-		(property "Reference" "R?"
+		(property "Reference" "R2"
 			(at 105.41 68.5799 0)
 			(effects
@@
 			(project "VOLK_enhanced_transmitter"
 				(path "/18397c79-8016-4b55-8616-aabd5bfb4047"
-					(reference "R?")
+					(reference "R2")
 					(unit 1)
 				)
@@
 		(dnp no)
 		(fields_autoplaced yes)
-		(property "Reference" "Q?"
+		(property "Reference" "Q1"
 			(at 116.84 62.2299 0)
 			(effects
@@
 			(project "VOLK_enhanced_transmitter"
 				(path "/18397c79-8016-4b55-8616-aabd5bfb4047"
-					(reference "Q?")
+					(reference "Q1")
 					(unit 1)
 				)
@@
 		(dnp no)
 		(fields_autoplaced yes)
-		(property "Reference" "R?"
-			(at 107.9118 44.45 0)
-			(effects
-				(font
-					(size 1.27 1.27)
-				)
-				(justify left)
+		(property "Reference" "R3"
+			(at 109.1819 40.64 90)
+			(effects
+				(font
+					(size 1.27 1.27)
+				)
 			)
 		)
 		(property "Value" "100k"
-			(at 110.4518 44.45 0)
-			(effects
-				(font
-					(size 1.27 1.27)
-				)
-				(justify left)
+			(at 109.1819 43.18 90)
+			(effects
+				(font
+					(size 1.27 1.27)
+				)
 			)
 		)
@@
 			(project "VOLK_enhanced_transmitter"
 				(path "/18397c79-8016-4b55-8616-aabd5bfb4047"
-					(reference "R?")
+					(reference "R3")
 					(unit 1)
 				)
@@
 		(dnp no)
 		(fields_autoplaced yes)
-		(property "Reference" "D?"
+		(property "Reference" "D1"
 			(at 117.7925 49.53 0)
 			(effects
@@
 			(project "VOLK_enhanced_transmitter"
 				(path "/18397c79-8016-4b55-8616-aabd5bfb4047"
-					(reference "D?")
-					(unit 1)
-				)
+					(reference "D1")
+					(unit 1)
+				)
